File: SFP_breakout.sch (KiCad schematic (older format))
At the start: 45 parts, among them J101 USB_B_Micro, J102 Conn_01x02, J103 Conn_02x02_Counter_Clockwise, J104 Conn_Coaxial, J105 Conn_Coaxial, J106 Conn_Coaxial, J107 Conn_Coaxial, P101 SFP-CONNECTOR, U101 LT1963AxQ-3.3, U102 74HC14

Commit message: add documentation to schematic
Parts:
- J101: symbol Connector:USB_B_Micro -> SFP_breakout-rescue:USB_B_Micro-Connector
- JP101: symbol Device:Jumper -> SFP_breakout-rescue:Jumper-Device
Other:
- note added: "TX_FAULT:\nshould be pulled up with a 4.7K – 10KΩ resistor on the host board. \nPull up voltage between 2.0V and VccT, R+0.3V. When high,output \nindicates a laser fault of some kind. Low indicates normal \noperation. In the lowstate, the output will be pulled to < 0.8V.\n\n\nTX_DISABLE\nLow (0 – 0.8V): Transmitter on\n(>0.8, < 2.0V): Undefined\nHigh (2.0 – 3.465V): Transmitter Disabled\nOpen: Tr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"
Changed lines of the file:
@@
 	6000 4600 6000 4550
 $Comp
-L Connector:USB_B_Micro J101
+L SFP_breakout-rescue:USB_B_Micro-Connector J101
 U 1 1 5BFF0CAB
 P 1100 5800
@@
 	5000 2500 4450 2500
 $Comp
-L Device:Jumper JP101
+L SFP_breakout-rescue:Jumper-Device JP101
 U 1 1 5C0A3EFC
 P 5150 1850
@@
 Text Notes 4650 6800 0    50   ~ 0
 1,9V 2mA LED\nuse 680R (?)
-Text Notes 2250 3950 0    50   ~ 0
+Text Notes 3000 4450 0    50   ~ 0
 describe rate-select here!
 $Comp
@@
 Wire Notes Line
 	7600 1450 7600 500
+Text Notes 700  4100 0    50   ~ 0
+TX_FAULT:\nshould be pulled up with a 4.7K – 10KΩ resistor on the host board. \nPull up voltage between 2.0V and VccT, R+0.3V.  When high,output \nindicates  a  laser  fault  of  some  kind.    Low  indicates  normal \noperation.  In  the  lowstate, the output will be pulled to < 0.8V.\n\n\nTX_DISABLE\nLow (0 – 0.8V):    Transmitter on\n(>0.8, < 2.0V):     Undefined\nHigh (2.0 – 3.465V): Transmitter Disabled\nOpen:                              Transmitter Disabled
 $EndSCHEMATC

Commit message: component values
Parts:
- C101, C103: value C -> 10u
- C102, C106, C107, C110, C111, C112, C113: value C -> 100n
- C104, C105: value C -> 1u
- C108, C109: value C -> 10n
- L101, L102: value L -> 1uH
- R101, R102, R103, R106: value R -> 680R
- R104, R105, R107, R108, R109: value 7k -> 6k8
Other:
- note added: "See SFP document\nINF-8074.PDF\nINF-8074i Specification for\nSFP (Small Formfactor Pluggable) Transceiver"
- note added: "TX_FAULT:\nshould be pulled up with a 4.7K – 10K resistor on the host board. \nPull up voltage between 2.0V and VccT, R+0.3V. When high,output \nindicates a laser fault of some kind. Low indicates normal \noperation. In the lowstate, the output will be pulled to < 0.8V.\n\n\nTX_DISABLE\nLow (0 – 0.8V): Transmitter on\n(>0.8, < 2.0V): Undefined\nHigh (2.0 – 3.465V): Transmitter Disabled\nOpen: Tra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"
- note added: "edge-mount SMA"
- note removed: "TX_FAULT:\nshould be pulled up with a 4.7K – 10KΩ resistor on the host board. \nPull up voltage between 2.0V and VccT, R+0.3V. When high,output \nindicates a laser fault of some kind. Low indicates normal \noperation. In the lowstate, the output will be pulled to < 0.8V.\n\n\nTX_DISABLE\nLow (0 – 0.8V): Transmitter on\n(>0.8, < 2.0V): Undefined\nHigh (2.0 – 3.465V): Transmitter Disabled\nOpen: Tr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"
Changed lines of the file:
@@
 P 2700 5800
 F 0 "C101" H 2815 5846 50  0000 L CNN
-F 1 "C" H 2815 5755 50  0000 L CNN
+F 1 "10u" H 2815 5755 50  0000 L CNN
 F 2 "Capacitor_SMD:C_0805_2012Metric" H 2738 5650 50  0001 C CNN
 F 3 "~" H 2700 5800 50  0001 C CNN
@@
 U 1 1 5BFF1966
 P 4450 5800
-F 0 "C103" H 4565 5846 50  0000 L CNN
-F 1 "C" H 4565 5755 50  0000 L CNN
+F 0 "C103" H 4150 5800 50  0000 L CNN
+F 1 "10u" H 4250 5700 50  0000 L CNN
 F 2 "Capacitor_SMD:C_0805_2012Metric" H 4488 5650 50  0001 C CNN
 F 3 "~" H 4450 5800 50  0001 C CNN
@@
 P 4750 6150
 F 0 "R106" H 4820 6196 50  0000 L CNN
-F 1 "R" H 4820 6105 50  0000 L CNN
+F 1 "680R" V 4750 6050 50  0000 L CNN
 F 2 "Resistor_SMD:R_0805_2012Metric" V 4680 6150 50  0001 C CNN
 F 3 "~" H 4750 6150 50  0001 C CNN
@@
 U 1 1 5BFF6D15
 P 7250 3500
-F 0 "C111" V 7300 3600 50  0000 C CNN
-F 1 "C" V 7200 3600 50  0000 C CNN
+F 0 "C111" V 7300 3650 50  0000 C CNN
+F 1 "100n" V 7300 3350 50  0000 C CNN
 F 2 "Capacitor_SMD:C_0805_2012Metric" H 7288 3350 50  0001 C CNN
 F 3 "~" H 7250 3500 50  0001 C CNN
@@
 U 1 1 5BFF6D83
 P 7250 3300
-F 0 "C110" V 7300 3400 50  0000 C CNN
-F 1 "C" V 7200 3400 50  0000 C CNN
+F 0 "C110" V 7300 3450 50  0000 C CNN
+F 1 "100n" V 7200 3150 50  0000 C CNN
 F 2 "Capacitor_SMD:C_0805_2012Metric" H 7288 3150 50  0001 C CNN
 F 3 "~" H 7250 3300 50  0001 C CNN
@@
 U 1 1 5BFF6F6F
 P 7250 4100
-F 0 "C113" V 7300 4200 50  0000 C CNN
-F 1 "C" V 7200 4200 50  0000 C CNN
+F 0 "C113" V 7300 4250 50  0000 C CNN
+F 1 "100n" V 7300 3950 50  0000 C CNN
 F 2 "Capacitor_SMD:C_0805_2012Metric" H 7288 3950 50  0001 C CNN
 F 3 "~" H 7250 4100 50  0001 C CNN
@@
 U 1 1 5BFF6F76
 P 7250 3900
-F 0 "C112" V 7300 4000 50  0000 C CNN
-F 1 "C" V 7200 4000 50  0000 C CNN
+F 0 "C112" V 7300 4050 50  0000 C CNN
+F 1 "100n" V 7200 3750 50  0000 C CNN
 F 2 "Capacitor_SMD:C_0805_2012Metric" H 7288 3750 50  0001 C CNN
 F 3 "~" H 7250 3900 50  0001 C CNN
@@
 U 1 1 5C009619
 P 6350 1700
-F 0 "C108" H 6465 1746 50  0000 L CNN
-F 1 "C" H 6465 1655 50  0000 L CNN
+F 0 "C108" H 6250 1950 50  0000 L CNN
+F 1 "10n" H 6465 1655 50  0000 L CNN
 F 2 "Capacitor_SMD:C_0805_2012Metric" H 6388 1550 50  0001 C CNN
 F 3 "~" H 6350 1700 50  0001 C CNN
@@
 U 1 1 5C00965F
 P 6150 1700
-F 0 "C106" H 6265 1746 50  0000 L CNN
-F 1 "C" H 6265 1655 50  0000 L CNN
+F 0 "C106" H 6050 1950 50  0000 L CNN
+F 1 "100n" H 6050 1600 50  0000 L CNN
 F 2 "Capacitor_SMD:C_0805_2012Metric" H 6188 1550 50  0001 C CNN
 F 3 "~" H 6150 1700 50  0001 C CNN
@@
 U 1 1 5C00969F
 P 5950 1700
-F 0 "C104" H 6065 1746 50  0000 L CNN
-F 1 "C" H 6065 1655 50  0000 L CNN
+F 0 "C104" H 5750 1800 50  0000 L CNN
+F 1 "1u" H 5750 1600 50  0000 L CNN
 F 2 "Capacitor_SMD:C_0805_2012Metric" H 5988 1550 50  0001 C CNN
 F 3 "~" H 5950 1700 50  0001 C CNN
@@
 P 5700 1500
 F 0 "L101" V 5522 1500 50  0000 C CNN
-F 1 "L" V 5613 1500 50  0000 C CNN
+F 1 "1uH" V 5613 1500 50  0000 C CNN
 F 2 "Inductor_SMD:L_0805_2012Metric" H 5700 1500 50  0001 C CNN
 F 3 "~" H 5700 1500 50  0001 C CNN
@@
 P 6350 2450
 F 0 "C109" H 6465 2496 50  0000 L CNN
-F 1 "C" H 6465 2405 50  0000 L CNN
+F 1 "10n" H 6465 2405 50  0000 L CNN
 F 2 "Capacitor_SMD:C_0805_2012Metric" H 6388 2300 50  0001 C CNN
 F 3 "~" H 6350 2450 50  0001 C CNN
@@
 U 1 1 5C01730C
 P 6150 2450
-F 0 "C107" H 6265 2496 50  0000 L CNN
-F 1 "C" H 6265 2405 50  0000 L CNN
+F 0 "C107" H 6050 2550 50  0000 L CNN
+F 1 "100n" H 6100 2350 50  0000 L CNN
 F 2 "Capacitor_SMD:C_0805_2012Metric" H 6188 2300 50  0001 C CNN
 F 3 "~" H 6150 2450 50  0001 C CNN
@@
 U 1 1 5C017313
 P 5950 2450
-F 0 "C105" H 6065 2496 50  0000 L CNN
-F 1 "C" H 6065 2405 50  0000 L CNN
+F 0 "C105" H 5700 2550 50  0000 L CNN
+F 1 "1u" H 5750 2350 50  0000 L CNN
 F 2 "Capacitor_SMD:C_0805_2012Metric" H 5988 2300 50  0001 C CNN
 F 3 "~" H 5950 2450 50  0001 C CNN
@@
 P 5700 2250
 F 0 "L102" V 5522 2250 50  0000 C CNN
-F 1 "L" V 5613 2250 50  0000 C CNN
+F 1 "1uH" V 5613 2250 50  0000 C CNN
 F 2 "Inductor_SMD:L_0805_2012Metric" H 5700 2250 50  0001 C CNN
 F 3 "~" H 5700 2250 50  0001 C CNN
@@
 P 4250 4300
 F 0 "R104" V 4150 4200 50  0000 L CNN
-F 1 "7k" V 4250 4250 50  0000 L CNN
+F 1 "6k8" V 4250 4250 50  0000 L CNN
 F 2 "Resistor_SMD:R_0805_2012Metric" V 4180 4300 50  0001 C CNN
 F 3 "~" H 4250 4300 50  0001 C CNN
@@
 P 4450 4300
 F 0 "R105" V 4550 4200 50  0000 L CNN
-F 1 "7k" V 4450 4250 50  0000 L CNN
+F 1 "6k8" V 4450 4250 50  0000 L CNN
 F 2 "Resistor_SMD:R_0805_2012Metric" V 4380 4300 50  0001 C CNN
 F 3 "~" H 4450 4300 50  0001 C CNN
@@
 U 1 1 5C042BDC
 P 4150 2500
-F 0 "U102" H 4150 2183 50  0000 C CNN
-F 1 "74HC14" H 4150 2274 50  0000 C CNN
+F 0 "U102" H 4350 2300 50  0000 C CNN
+F 1 "74HC14" H 4350 2400 50  0000 C CNN
 F 2 "Package_SO:TSSOP-14_4.4x5mm_P0.65mm" H 4150 2500 50  0001 C CNN
 F 3 "http://www.ti.com/lit/gpn/sn74HC14" H 4150 2500 50  0001 C CNN
@@
 U 2 1 5C042CD1
 P 4150 2800
-F 0 "U102" H 4150 2483 50  0000 C CNN
-F 1 "74HC14" H 4150 2574 50  0000 C CNN
+F 0 "U102" H 4350 2600 50  0000 C CNN
+F 1 "74HC14" H 4350 2700 50  0000 C CNN
 F 2 "Package_SO:TSSOP-14_4.4x5mm_P0.65mm" H 4150 2800 50  0001 C CNN
 F 3 "http://www.ti.com/lit/gpn/sn74HC14" H 4150 2800 50  0001 C CNN
@@
 U 3 1 5C042DB5
 P 4150 3100
-F 0 "U102" H 4150 2783 50  0000 C CNN
-F 1 "74HC14" H 4150 2874 50  0000 C CNN
+F 0 "U102" H 4350 2900 50  0000 C CNN
+F 1 "74HC14" H 4300 3000 50  0000 C CNN
 F 2 "Package_SO:TSSOP-14_4.4x5mm_P0.65mm" H 4150 3100 50  0001 C CNN
 F 3 "http://www.ti.com/lit/gpn/sn74HC14" H 4150 3100 50  0001 C CNN
@@
 U 1 1 5C04B2A3
 P 3500 1500
-F 0 "C102" H 3615 1546 50  0000 L CNN
-F 1 "C" H 3615 1455 50  0000 L CNN
+F 0 "C102" H 3500 1600 50  0000 L CNN
+F 1 "100n" H 3500 1400 50  0000 L CNN
 F 2 "Capacitor_SMD:C_0805_2012Metric" H 3538 1350 50  0001 C CNN
 F 3 "~" H 3500 1500 50  0001 C CNN
@@
 U 1 1 5C053B18
 P 2950 2300
-F 0 "D102" V 2988 2183 50  0000 R CNN
-F 1 "LED" V 2897 2183 50  0000 R CNN
+F 0 "D102" V 3000 2600 50  0000 R CNN
+F 1 "LED" V 2900 2600 50  0000 R CNN
 F 2 "LED_SMD:LED_0805_2012Metric" H 2950 2300 50  0001 C CNN
 F 3 "~" H 2950 2300 50  0001 C CNN
@@
 U 1 1 5C053D26
 P 2950 1950
-F 0 "R101" H 3020 1996 50  0000 L CNN
-F 1 "R" H 3020 1905 50  0000 L CNN
+F 0 "R101" V 3000 1650 50  0000 L CNN
+F 1 "680R" V 2950 1850 50  0000 L CNN
 F 2 "Resistor_SMD:R_0805_2012Metric" V 2880 1950 50  0001 C CNN
 F 3 "~" H 2950 1950 50  0001 C CNN
@@
 U 1 1 5C053DD4
 P 3150 1950
-F 0 "R102" H 3220 1996 50  0000 L CNN
-F 1 "R" H 3220 1905 50  0000 L CNN
+F 0 "R102" V 3200 1650 50  0000 L CNN
+F 1 "680R" V 3150 1850 50  0000 L CNN
 F 2 "Resistor_SMD:R_0805_2012Metric" V 3080 1950 50  0001 C CNN
 F 3 "~" H 3150 1950 50  0001 C CNN
@@
 U 1 1 5C053E36
 P 3350 1950
-F 0 "R103" H 3420 1996 50  0000 L CNN
-F 1 "R" H 3420 1905 50  0000 L CNN
+F 0 "R103" V 3400 1650 50  0000 L CNN
+F 1 "680R" V 3350 1850 50  0000 L CNN
 F 2 "Resistor_SMD:R_0805_2012Metric" V 3280 1950 50  0001 C CNN
 F 3 "~" H 3350 1950 50  0001 C CNN
@@
 P 5000 2250
 F 0 "R109" V 5000 2450 50  0000 L CNN
-F 1 "7k" V 5000 2200 50  0000 L CNN
+F 1 "6k8" V 5000 2200 50  0000 L CNN
 F 2 "Resistor_SMD:R_0805_2012Metric" V 4930 2250 50  0001 C CNN
 F 3 "~" H 5000 2250 50  0001 C CNN
@@
 P 4900 2250
 F 0 "R108" V 4900 2450 50  0000 L CNN
-F 1 "7k" V 4900 2200 50  0000 L CNN
+F 1 "6k8" V 4900 2200 50  0000 L CNN
 F 2 "Resistor_SMD:R_0805_2012Metric" V 4830 2250 50  0001 C CNN
 F 3 "~" H 4900 2250 50  0001 C CNN
@@
 P 4800 2250
 F 0 "R107" V 4800 2450 50  0000 L CNN
-F 1 "7k" V 4800 2200 50  0000 L CNN
+F 1 "6k8" V 4800 2200 50  0000 L CNN
 F 2 "Resistor_SMD:R_0805_2012Metric" V 4730 2250 50  0001 C CNN
 F 3 "~" H 4800 2250 50  0001 C CNN
@@
 	7600 1450 7600 500
 Text Notes 700  4100 0    50   ~ 0
-TX_FAULT:\nshould be pulled up with a 4.7K – 10KΩ resistor on the host board. \nPull up voltage between 2.0V and VccT, R+0.3V.  When high,output \nindicates  a  laser  fault  of  some  kind.    Low  indicates  normal \noperation.  In  the  lowstate, the output will be pulled to < 0.8V.\n\n\nTX_DISABLE\nLow (0 – 0.8V):    Transmitter on\n(>0.8, < 2.0V):     Undefined\nHigh (2.0 – 3.465V): Transmitter Disabled\nOpen:                              Transmitter Disabled
+TX_FAULT:\nshould be pulled up with a 4.7K – 10K resistor on the host board. \nPull up voltage between 2.0V and VccT, R+0.3V.  When high,output \nindicates  a  laser  fault  of  some  kind.    Low  indicates  normal \noperation.  In  the  lowstate, the output will be pulled to < 0.8V.\n\n\nTX_DISABLE\nLow (0 – 0.8V):    Transmitter on\n(>0.8, < 2.0V):     Undefined\nHigh (2.0 – 3.465V): Transmitter Disabled\nOpen:                              Transmitter Disabled
+Text Notes 8500 3600 0    50   ~ 0
+edge-mount SMA
+Text Notes 7750 2050 0    50   ~ 0
+See SFP document\nINF-8074.PDF\nINF-8074i Specification for\nSFP (Small Formfactor Pluggable) Transceiver
 $EndSCHEMATC

Commit message: add notes
Other:
- note added: "Digikey 296-8234-1-ND\n"
- note added: "Digikey A98333-ND\n"
- note added: "connector Digikey A97943CT-ND\ncage U77-A1114-100TCT-ND\n\n"
- note added: "edge-mount SMA\nDigikey ACX1426-ND\n"
- note removed: "edge-mount SMA"
Changed lines of the file:
@@
 TX_FAULT:\nshould be pulled up with a 4.7K – 10K resistor on the host board. \nPull up voltage between 2.0V and VccT, R+0.3V.  When high,output \nindicates  a  laser  fault  of  some  kind.    Low  indicates  normal \noperation.  In  the  lowstate, the output will be pulled to < 0.8V.\n\n\nTX_DISABLE\nLow (0 – 0.8V):    Transmitter on\n(>0.8, < 2.0V):     Undefined\nHigh (2.0 – 3.465V): Transmitter Disabled\nOpen:                              Transmitter Disabled
 Text Notes 8500 3600 0    50   ~ 0
-edge-mount SMA
+edge-mount SMA\nDigikey ACX1426-ND\n
 Text Notes 7750 2050 0    50   ~ 0
 See SFP document\nINF-8074.PDF\nINF-8074i Specification for\nSFP (Small Formfactor Pluggable) Transceiver
+Text Notes 5450 3000 0    50   ~ 0
+connector Digikey A97943CT-ND\ncage U77-A1114-100TCT-ND\n\n
+Text Notes 4000 1350 0    50   ~ 0
+Digikey 296-8234-1-ND\n
+Text Notes 450  5050 0    50   ~ 0
+Digikey A98333-ND\n
 $EndSCHEMATC
