File: SFP_breakout.kicad_pcb (KiCad board)
At the start: 2 copper layers, 100 x 70 mm, 47 parts, among them J101 USB_B_Micro, J102 Conn_01x02, J103 Conn_02x02_Counter_Clockwise, J104 Conn_Coaxial, J105 Conn_Coaxial, J106 Conn_Coaxial, J107 Conn_Coaxial, P101 SFP-CONNECTOR, U101 LT1963AxQ-3.3, U102 74HC14

Commit message: PCB order ca 2021-06-01
Other:
- rule pad_to_mask_clearance: 0.051 -> 0

Commit message: kicad7 version
Other:
- net class Default removed
